File: PMU_HW.kicad_pcb (KiCad board)
At the start: 2 copper layers, 9 parts, among them J1 Conn_01x08_Male, J2 Conn_01x08_Male, J3 Conn_01x02_Female, U2 ADS8681IPWR

Commit message: lul
Parts:
- moved C4 64.6 mm to (107.3, 78.0)
- moved C1 50.9 mm to (100.6, 70.0), turned to 180 degrees
- moved C3 48.3 mm to (103.5, 69.1), turned to 90 degrees
- moved J2 46.6 mm to (108.3, 83.1)
- moved C2 45.8 mm to (100.6, 68.2), turned to 180 degrees
- moved C5 45.1 mm to (106.3, 70.2)
- moved J3 43.9 mm to (112.4, 73.0)
- moved U2 42.7 mm to (102.7, 74.9), turned to 270 degrees
- moved J1 28.9 mm to (108.3, 65.3), turned to 270 degrees
Connections:
- J1 pad 1: Net-(J1-Pad1) -> GNDA
- J1 pad 2: Net-(J1-Pad2) -> /ALARM
- J1 pad 4: Net-(J1-Pad4) -> +3V3
- J1 pad 6: Net-(J1-Pad6) -> GNDA
- J1 pad 8: Net-(J1-Pad8) -> +5VA
- J2 pad 1: Net-(J2-Pad1) -> GNDA
- J2 pad 2: Net-(J2-Pad2) -> /RVS
- J2 pad 3: Net-(J2-Pad3) -> /SDO
- J2 pad 4: Net-(J2-Pad4) -> /SDI
- J2 pad 5: Net-(J2-Pad5) -> /SCLK
- J2 pad 6: Net-(J2-Pad6) -> GNDA
- J2 pad 7: Net-(J2-Pad7) -> /CS
- J2 pad 8: Net-(J2-Pad8) -> /RST
- U2 pad 10: /SCLK -> /SDI
- U2 pad 11: /SDO -> /CS
- U2 pad 12: /ALARM -> /SCLK
- U2 pad 13: /RVS -> /SDO
- U2 pad 14: +3V3 -> /ALARM
- U2 pad 15: GNDA -> /RVS
- U2 pad 16: +5VA -> +3V3
- U2 pad 2: /REF_O -> +5VA
- U2 pad 4: /REF_CAP -> /REF_O
- U2 pad 5: Net-(J3-Pad2) -> GNDA
- U2 pad 6: GNDA -> /REF_CAP
- U2 pad 7: /RST -> Net-(J3-Pad2)
- U2 pad 8: /SDI -> GNDA
- U2 pad 9: /CS -> /RST
Routing:
- net /SDO: track 0.00 -> 13.7 mm, vias 0 -> 1
- net /RST: track 0.00 -> 13.4 mm
- net Net-(J3-Pad2): track 0.00 -> 13.1 mm
- net /CS: track 0.00 -> 12.4 mm
- net /SDI: track 0.00 -> 11.7 mm, vias 0 -> 1
- net /SCLK: track 0.00 -> 11.0 mm, vias 0 -> 1
- net /RVS: track 0.00 -> 5.80 mm
- net +5VA: track 0.00 -> 2.27 mm
- net /REF_CAP: track 2.33 -> 3.99 mm
- net +3V3: track 0.00 -> 1.51 mm
- net GNDA: track 0.79 -> 0.00 mm
- added copper zone on F.Cu, net GNDA
Other:
- board outline added: 34.2 x 21.5 mm

Commit message: finished
Parts:
- added C6: 2u2, Capacitor_SMD:C_0603_1608Metric_Pad1.08x0.95mm_HandSolder, F.Cu at (149.5, 115.5)
- moved C2 69.7 mm to (155.3, 111.4), turned to 0 degrees
- moved C1 67.2 mm to (152.5, 112.6), turned to 270 degrees
- moved J1 66.2 mm to (148.0, 118.4), turned to 90 degrees
- moved C3 64.0 mm to (150.5, 112.6), turned to 270 degrees
- moved C5 58.5 mm to (147.8, 111.4), turned to 180 degrees
- moved U2 57.8 mm to (151.0, 106.7), turned to 90 degrees
- moved J3 56.4 mm to (158.0, 106.2)
- moved C4 48.0 mm to (147.3, 104.5), turned to 270 degrees
- moved J2 43.3 mm to (148.0, 100.6), turned to 90 degrees
Connections:
- J1 pad 1: GNDA -> +5VA
- J1 pad 2: /ALARM -> GNDA
- J1 pad 3: Net-(J1-Pad3) -> +3V3
- J1 pad 4: +3V3 -> Net-(J1-Pad4)
- J1 pad 6: GNDA -> Net-(J1-Pad6)
- J1 pad 8: +5VA -> GNDA
- J2 pad 1: GNDA -> /SDO
- J2 pad 2: /RVS -> Net-(J2-Pad2)
- J2 pad 3: /SDO -> /SCLK
- J2 pad 5: /SCLK -> /RST
- J2 pad 6: GNDA -> /CS
- J2 pad 7: /CS -> /ALARM
- J2 pad 8: /RST -> /RVS
Routing:
- net GNDA: track 0.00 -> 24.2 mm, vias 0 -> 4
- net +3V3: track 1.51 -> 21.1 mm, vias 0 -> 1
- net /ALARM: track 0.00 -> 16.9 mm
- net /RVS: track 5.80 -> 20.5 mm
- net /SDO: track 13.7 -> 4.49 mm, vias 1 -> 0
- net /RST: track 13.4 -> 6.18 mm
- net +5VA: track 2.27 -> 9.41 mm
- net /SCLK: track 11.0 -> 3.94 mm, vias 1 -> 0
- net /SDI: track 11.7 -> 5.27 mm, vias 1 -> 0
- net Net-(J3-Pad2): track 13.1 -> 6.81 mm
- net /CS: track 12.4 -> 11.3 mm
- added copper zone on B.Cu, net GNDA
Other:
- board size 34.2 x 21.5 mm -> 21.5 x 21.5 mm
- net class Power added: clearance 0.2, trace_width 0.5, via_dia 0.8, via_drill 0.4

Commit message: clean up
Other:
- net class Default removed
- net class Power removed
